File: hardware/EthCtrlMeter.brd (EAGLE design)
At the start: 86.4 x 31.7 mm, 66 parts, among them IC1 ESP32-WROOM-32D_M113DH3200PH3Q, IC2 LAN8720A-CP-ABC, IC3 R-78E3.3-1.0, J2 1727078, J3 HR911105A, J4 1727010, Q1 O50.0-JO32-B-3.3-1

Commit message: update
Parts:
- R23, R29: value 27R -> DNP
- R31: value 27R -> 33R
Changed lines of the file:
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@@
 <drawing>
 <settings>
-<setting alwaysvectorfont="yes"/>
+<setting alwaysvectorfont="no"/>
 <setting verticaltext="up"/>
 </settings>
@@
 </layers>
 <board>
-<fusionsync huburn="a.cGVyc29uYWw6dWUyYzBhZTFk" projecturn="a.cGVyc29uYWw6dWUyYzBhZTFkIzIwMjEwNDE3NDAzOTg2MzA2" f3durn="urn:adsk.wipprod:dm.lineage:QqtcW-pHTzKlH9XkH0GQuw" pcbguid="" lastpulledtime="2022-01-10T20:19:45Z" lastsyncedchangeguid="" latestrevisionid="7b5390ac-47e2-4a57-a6a9-9916ae84fb58" lastsyncedrevisionid="7b5390ac-47e2-4a57-a6a9-9916ae84fb58" lastboardhashguid="d29f7d26-245f-ad2a-6957-bbebb5ddb7d6" lastpushedtime="2022-01-10T20:43:02Z" linktopcb3d="true"/>
+<fusionsync huburn="a.cGVyc29uYWw6dWUyYzBhZTFk" projecturn="a.cGVyc29uYWw6dWUyYzBhZTFkIzIwMjEwNDE3NDAzOTg2MzA2" f3durn="urn:adsk.wipprod:dm.lineage:QqtcW-pHTzKlH9XkH0GQuw" pcbguid="" lastpulledtime="2022-01-10T20:19:45Z" lastsyncedchangeguid="" latestrevisionid="7b5390ac-47e2-4a57-a6a9-9916ae84fb58" lastsyncedrevisionid="7b5390ac-47e2-4a57-a6a9-9916ae84fb58" lastboardhashguid="d29f7d26-245f-ad2a-6957-bbebb5ddb7d6" lastpushedtime="2022-01-10T20:43:02Z" linktopcb3d="false"/>
 <plain>
 <polygon width="0.1524" layer="39">
@@
 <attribute name="VALUE" x="51.535" y="7.905" size="1.27" layer="27" rot="R180"/>
 </element>
-<element name="R23" library="rcl" library_urn="urn:adsk.eagle:library:334" package="R0603" package3d_urn="urn:adsk.eagle:package:23555/3" value="27R" x="50.9" y="10.1" smashed="yes">
+<element name="R23" library="rcl" library_urn="urn:adsk.eagle:library:334" package="R0603" package3d_urn="urn:adsk.eagle:package:23555/3" value="DNP" x="50.9" y="10.1" smashed="yes">
 <attribute name="NAME" x="52.465" y="9.935" size="0.8128" layer="25"/>
 <attribute name="POPULARITY" value="70" x="50.9" y="10.1" size="1.778" layer="27" display="off"/>
@@
 <attribute name="VALUE" x="55.835" y="9.295" size="1.27" layer="28" rot="MR0"/>
 </element>
-<element name="R29" library="rcl" library_urn="urn:adsk.eagle:library:334" package="R0603" package3d_urn="urn:adsk.eagle:package:23555/3" value="27R" x="59.9" y="4.6" smashed="yes" rot="MR270">
+<element name="R29" library="rcl" library_urn="urn:adsk.eagle:library:334" package="R0603" package3d_urn="urn:adsk.eagle:package:23555/3" value="DNP" x="59.9" y="4.6" smashed="yes" rot="MR270">
 <attribute name="NAME" x="58.465" y="2.965" size="0.8128" layer="26" rot="MR180"/>
 <attribute name="POPULARITY" value="70" x="59.9" y="4.6" size="1.778" layer="28" rot="MR270" display="off"/>
@@
 <attribute name="VALUE" x="8.5" y="2.7" size="1.27" layer="27" rot="R270" align="center"/>
 </element>
-<element name="R31" library="rcl" library_urn="urn:adsk.eagle:library:334" package="R0603" package3d_urn="urn:adsk.eagle:package:23555/3" value="27R" x="50.9" y="12.1" smashed="yes">
+<element name="R31" library="rcl" library_urn="urn:adsk.eagle:library:334" package="R0603" package3d_urn="urn:adsk.eagle:package:23555/3" value="33R" x="50.9" y="12.1" smashed="yes">
 <attribute name="NAME" x="49.565" y="12.835" size="0.8128" layer="25"/>
 <attribute name="POPULARITY" value="70" x="50.9" y="12.1" size="1.778" layer="27" display="off"/>
